Commit message: Post Lab3 Updates

File: urdf/robot.xacro (robot description, xacro)
@@ -1,150 +1,66 @@
 <?xml version="1.0"?>
 <robot xmlns:xacro="http://www.ros.org/wiki/xacro" name="navvis">
-	<link name="base">
-		<visual>
-			<!-- Shift the box up half its height. !-->
-			<origin xyz="0.0 0.0 0.96" rpy="0.0 0.0 0.0" />
-			<geometry>
-				<box size="0.45 0.78 1.92" />
-			</geometry>
-		</visual>
-		<collision>
-			<!-- Shift the box up half its height. !-->
-			<origin xyz="0.0 0.0 0.96" rpy="0.0 0.0 0.0" />
-			<geometry>
-				<box size="0.45 0.78 1.92" />
-			</geometry>
-		</collision>
-	</link>
-	<link name="laser_vert_bottom_joint">
-		<visual>
-			<geometry>
-				<box size="0.062 0.062 0.087" />
-			</geometry>
-		</visual>
-		<collision>
-			<geometry>
-				<box size="0.062 0.062 0.087" />
-			</geometry>
-		</collision>
-	</link>
-	<joint name="base_laser_vert_bottom_joint" type="fixed">
-		<parent link="base" />
-		<child link="laser_vert_bottom_joint" />
-		<origin xyz="0.3158 -0.0021 0.5100" rpy="3.1355 -1.3045 0.0025" />
-	</joint>
-	<link name="laser_vert_top_right_joint">
-		<visual>
-			<geometry>
-				<box size="0.062 0.062 0.087" />
-			</geometry>
-		</visual>
-		<collision>
-			<geometry>
-				<box size="0.062 0.062 0.087" />
-			</geometry>
-		</collision>
-	</link>
-	<joint name="base_laser_vert_top_right_joint" type="fixed">
-		<parent link="base" />
-		<child link="laser_vert_top_right_joint" />
-		<origin xyz="0.2978 -0.1450 1.8451" rpy="-1.1760 0.6313 -1.9377" />
-	</joint>
-	<link name="laser_vert_top_left_joint">
-		<visual>
-			<geometry>
-				<box size="0.062 0.062 0.087" />
-			</geometry>
-		</visual>
-		<collision>
-			<geometry>
-				<box size="0.062 0.062 0.087" />
-			</geometry>
-		</collision>
-	</link>
-	<joint name="base_laser_vert_top_left_joint" type="fixed">
-		<parent link="base" />
-		<child link="laser_vert_top_left_joint" />
-		<origin xyz="0.2997 0.1531 1.8443" rpy="1.1780 0.6198 1.9560" />
-	</joint>
-	<link name="laser_horiz_joint">
-		<visual>
-			<geometry>
-				<cylinder radius="0.052" length = "0.072" />
-			</geometry>
-		</visual>
-		<collision>
-			<geometry>
-				<cylinder radius="0.052" length = "0.072" />
-			</geometry>
-		</collision>
-	</link>
-	<joint name="base_laser_horiz_joint" type="fixed">
-		<parent link="base" />
-		<child link="laser_horiz_joint" />
-		<origin xyz="0.2325 0.0001 1.9201" rpy="-0.0012 0.1146 -0.0015" />
-	</joint>
-	<link name="wheel_left_joint">
-		<visual>
-			<geometry>
-				<cylinder radius="0.2" length = "0.05" />
-			</geometry>
-		</visual>
-		<collision>
-			<geometry>
-				<cylinder radius="0.2" length = "0.05" />
-			</geometry>
-		</collision>
-	</link>
-	<joint name="base_wheel_left_joint" type="continuous">
-		<parent link="base" />
-		<child link="wheel_left_joint" />
-		<origin xyz="0.10 0.4 0.0" rpy="-1.57079 0.0 0.0" />
-		<limit  effort="30" velocity="1.0" lower="-2.2" upper="0.7" />
-		<axis xyz="0.0 0.0 1.0"/>
-	</joint>
-	<link name="wheel_right_joint">
-		<visual>
-			<geometry>
-				<cylinder radius="0.2" length = "0.05" />
-			</geometry>
-		</visual>
-		<collision>
-			<geometry>
-				<cylinder radius="0.2" length = "0.05" />
-			</geometry>
-		</collision>
-	</link>
-	<joint name="base_wheel_right_joint" type="continuous">
-		<parent link="base" />
-		<child link="wheel_right_joint" />
-		<origin xyz="0.10 -0.4 0.0" rpy="-1.57079 0.0 0.0" />
-		<limit  effort="30" velocity="1.0" lower="-2.2" upper="0.7" />
-		<axis xyz="0.0 0.0 1.0"/>
-	</joint>
-	<link name="wheel_center_joint">
-		<visual>
-			<geometry>
-				<cylinder radius="0.15" length = "0.05" />
-			</geometry>
-		</visual>
-		<collision>
-			<geometry>
-				<cylinder radius="0.15" length = "0.05" />
-			</geometry>
-		</collision>
-	</link>
-	<joint name="base_wheel_center_joint" type="continuous">
-		<parent link="base" />
-		<child link="wheel_center_joint" />
-		<origin xyz="0.10 0.0 0.0" rpy="-1.57079 0.0 0.0" />
-		<limit  effort="30" velocity="1.0" lower="-2.2" upper="0.7" />
-		<axis xyz="0.0 0.0 1.0"/>
-	</joint>
-	<xacro:include filename="$(find gazebo_plugins)/test/multi_robot_scenario/xacro/laser/hokuyo.xacro" />
-  	<xacro:laser name="gazebo_laser_vert_bottom" parent="base" xyz="0.3157894464801903 -0.002068548615034871 0.5099999434059285" rpy="3.1354753 -1.3045001 		0.0024658" meshes="package://gazebo_plugins/test/multi_robot_scenario/meshes/laser" />
-  	<xacro:include filename="$(find velodyne_description)/urdf/VLP-16.urdf.xacro"/>
-  	<xacro:VLP-16 parent="base" name="gazebo_laser_horiz" topic="laser_horiz/packets" hz="10" samples="440" gpu="false">
-    	<origin xyz="0.2325416305773505 -0.0001380069427607134 1.920122926231907" rpy="-0.0012068 0.114646 -0.0015308" />
-  	</xacro:VLP-16>
-</robot>
+    <link name="base">
+    <visual>
+      <origin xyz="0.0 0.0 0.96" rpy="0.0 0.0 0.0" />
+      <geometry>
+        <box size="0.45 0.78 1.92" />
+      </geometry>
+    </visual>
+    <collision>
+      <origin xyz="0.0 0.0 0.96" rpy="0.0 0.0 0.0" />
+      <geometry>
+        <box size="0.45 0.78 1.92" />
+      </geometry>
+    </collision>
+  </link>
+  <xacro:macro name="side_wheels" params="side reflect">
+    <link name="wheel_${side}">
+      <visual>
+        <geometry>
+          <cylinder radius="0.2" length="0.05"/>
+        </geometry>
+      </visual>
+      <collision>
+        <geometry>
+          <cylinder radius="0.2" length="0.05"/>
+        </geometry>
+      </collision>
+    </link>
+    <joint name="base_wheel_${side}_joint" type="continuous">
+      <parent link="base" />
+      <child link="wheel_${side}" />
+      <origin xyz="-0.10 ${reflect * 0.4} 0.0" rpy="${-pi/2} 0.0 0.0" />
+      <axis xyz="0.0 0.0 1.0" />
+    </joint>
+  </xacro:macro>
+  <xacro:side_wheels side="left" reflect="1" />
+  <xacro:side_wheels side="right" reflect="-1" />
+  <link name="wheel_center">
+    <visual>
+      <geometry>
+        <cylinder radius="0.15" length="0.05"/>
+      </geometry>
+    </visual>
+    <collision>
+      <geometry>
+        <cylinder radius="0.15" length="0.05"/>
+      </geometry>
+    </collision>
+  </link>
+  <joint name="base_wheel_center_joint" type="continuous">
+    <parent link="base" />
+    <child link="wheel_center" />
+    <origin xyz="0.10 0.0 -0.05" rpy="${-pi/2} 0.0 0.0" />
+    <axis xyz="0.0 0.0 1.0" />
+  </joint>
+  <xacro:include filename="$(find gazebo_plugins)/test/multi_robot_scenario/xacro/laser/hokuyo.xacro" />
+  <xacro:laser name="gazebo_laser_vert_bottom" parent="base" xyz="0.3157894464801903 -0.002068548615034871 0.5099999434059285" rpy="3.1354753 -1.3045001 0.0024658" meshes="package://gazebo_plugins/test/multi_robot_scenario/meshes/laser" />
+  <xacro:laser name="laser_vert_bottom" parent="base" xyz="0.3157894464801903 -0.002068548615034871 0.5099999434059285" rpy="3.1354753 -1.3045001 0.0024658" meshes="package://gazebo_plugins/test/multi_robot_scenario/meshes/laser" />
+    <xacro:laser name="laser_vert_top_left" parent="base" xyz="0.2997 0.1531 1.8443" rpy="1.1780 0.6198 1.9560" meshes="package://gazebo_plugins/test/multi_robot_scenario/meshes/laser" />
+    <xacro:laser name="laser_vert_top_right" parent="base" xyz="0.2978 -0.1450 1.8451" rpy="-1.1760 0.6313 -1.9377" meshes="package://gazebo_plugins/test/multi_robot_scenario/meshes/laser" />
+  <xacro:include filename="$(find velodyne_description)/urdf/VLP-16.urdf.xacro"/>
+  <xacro:VLP-16 parent="base" name="laser_horiz" topic="laser_horiz/packets" hz="10" samples="440" gpu="false">
+    <origin xyz="0.2325416305773505 -0.0001380069427607134 1.920122926231907" rpy="-0.0012068 0.114646 -0.0015308" />
+  </xacro:VLP-16>
+ </robot>
